File: HB-MOD-UART/HB-MOD-UART.kicad_pcb (KiCad board)
At the start: 2 copper layers, 50 x 17.8 mm, 8 parts, among them J1 Conn_Raspi, J2 Conn_Coaxial, U1 HM-MOD-UART

Commit message: HB-MOD-UART: swap RX/TX
fixes #3
Connections:
- U1 pad 5: Net-(R1-Pad1) -> Net-(R2-Pad1)
- U1 pad 6: Net-(R2-Pad1) -> Net-(R1-Pad1)
Routing:
- net Net-(R2-Pad1): track 3.92 -> 3.09 mm
- net Net-(R1-Pad1): track 2.92 -> 3.75 mm
Other:
- board text added: "stan23 Nov 2019 V1.1 CC BY-NC-SA"
- board text removed: "stan23 Nov 2019 V1.0 CC BY-NC-SA"
Changed lines of the file:
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@@
   )
   (setup
-    (last_trace_width 0.3)
+    (last_trace_width 0.5)
     (user_trace_width 0.3)
     (user_trace_width 0.5)
@@
       (net 3 "Net-(J1-Pad12)"))
     (pad 5 thru_hole circle (at -3 -2 270) (size 1.27 1.27) (drill 0.762) (layers *.Cu *.Mask)
+      (net 9 "Net-(R2-Pad1)"))
+    (pad 6 thru_hole oval (at -5 -2 270) (size 1.27 1.27) (drill 0.762) (layers *.Cu *.Mask)
       (net 8 "Net-(R1-Pad1)"))
-    (pad 6 thru_hole oval (at -5 -2 270) (size 1.27 1.27) (drill 0.762) (layers *.Cu *.Mask)
-      (net 9 "Net-(R2-Pad1)"))
     (pad 1 smd rect (at 5 -2 270) (size 1.2 5) (layers F.Cu F.Mask)
       (net 1 +3V3))
@@
       (net 3 "Net-(J1-Pad12)"))
     (pad 5 smd rect (at -3 -2 270) (size 1.2 5) (layers F.Cu F.Mask)
+      (net 9 "Net-(R2-Pad1)"))
+    (pad 6 smd rect (at -5 -2 270) (size 1.2 5) (layers F.Cu F.Mask)
       (net 8 "Net-(R1-Pad1)"))
-    (pad 6 smd rect (at -5 -2 270) (size 1.2 5) (layers F.Cu F.Mask)
-      (net 9 "Net-(R2-Pad1)"))
     (pad 9 smd rect (at -2.5 -26.5 270) (size 1.5 4) (layers F.Cu F.Mask)
       (net 4 "Net-(J2-Pad1)"))
@@
     (effects (font (size 1 1) (thickness 0.15)))
   )
-  (gr_text "stan23\nNov 2019\nV1.0\nCC BY-NC-SA" (at 90.424 106.172 90) (layer B.SilkS)
+  (gr_text "stan23\nNov 2019\nV1.1\nCC BY-NC-SA" (at 90.424 106.172 90) (layer B.SilkS)
     (effects (font (size 1 1) (thickness 0.15)) (justify mirror))
   )
@@
   (gr_line (start 63.5 96.52) (end 113.538 96.52) (layer Edge.Cuts) (width 0.05))
   (gr_line (start 63.5 114.3) (end 63.5 96.52) (layer Edge.Cuts) (width 0.05))
-  (segment (start 72.624 111.76) (end 73.152 111.232) (width 0.5) (layer B.Cu) (net 1))
-  (segment (start 68.58 111.76) (end 72.624 111.76) (width 0.5) (layer B.Cu) (net 1))
-  (segment (start 75.092 111.232) (end 75.914 110.41) (width 0.5) (layer B.Cu) (net 1))
-  (segment (start 73.152 111.232) (end 75.092 111.232) (width 0.5) (layer B.Cu) (net 1))
-  (segment (start 80.828 110.41) (end 81.28 110.862) (width 0.5) (layer B.Cu) (net 1))
-  (segment (start 79.812 110.41) (end 80.264 110.862) (width 0.5) (layer B.Cu) (net 1))
-  (segment (start 75.914 110.41) (end 79.812 110.41) (width 0.5) (layer B.Cu) (net 1))
+  (segment (start 72.624 111.76) (end 73.152 111.232) (width 0.5) (layer B.Cu) (net 1) (status 30))
+  (segment (start 68.58 111.76) (end 72.624 111.76) (width 0.5) (layer B.Cu) (net 1) (status 30))
+  (segment (start 75.092 111.232) (end 75.914 110.41) (width 0.5) (layer B.Cu) (net 1) (status 20))
+  (segment (start 73.152 111.232) (end 75.092 111.232) (width 0.5) (layer B.Cu) (net 1) (status 10))
+  (segment (start 80.828 110.41) (end 81.28 110.862) (width 0.5) (layer B.Cu) (net 1) (status 30))
+  (segment (start 79.812 110.41) (end 80.264 110.862) (width 0.5) (layer B.Cu) (net 1) (status 30))
+  (segment (start 75.914 110.41) (end 79.812 110.41) (width 0.5) (layer B.Cu) (net 1) (status 30))
   (segment (start 67.31 102.87) (end 64.77 102.87) (width 0.3) (layer B.Cu) (net 2))
-  (segment (start 68.58 101.6) (end 67.31 102.87) (width 0.3) (layer B.Cu) (net 2))
+  (segment (start 68.58 101.6) (end 67.31 102.87) (width 0.3) (layer B.Cu) (net 2) (status 10))
   (via (at 64.77 102.87) (size 0.8) (drill 0.4) (layers F.Cu B.Cu) (net 2))
   (segment (start 66.04 99.06) (end 67.379999 100.399999) (width 0.3) (layer F.Cu) (net 3) (status 10))
   (segment (start 67.379999 100.399999) (end 69.156001 100.399999) (width 0.3) (layer F.Cu) (net 3))
-  (segment (start 75.914 104.41) (end 71.898 104.41) (width 0.5) (layer F.Cu) (net 3))
+  (segment (start 75.914 104.41) (end 71.898 104.41) (width 0.5) (layer F.Cu) (net 3) (status 10))
   (segment (start 71.898 104.41) (end 71.12 103.632) (width 0.5) (layer F.Cu) (net 3))
   (segment (start 71.12 103.632) (end 71.12 101.6) (width 0.5) (layer F.Cu) (net 3))
   (segment (start 71.12 101.6) (end 69.919999 100.399999) (width 0.5) (layer F.Cu) (net 3))
   (segment (start 69.156001 100.399999) (end 69.919999 100.399999) (width 0.3) (layer F.Cu) (net 3))
-  (segment (start 101.664 102.91) (end 100.414 102.91) (width 0.5) (layer F.Cu) (net 4))
-  (segment (start 108.458 105.41) (end 104.164 105.41) (width 0.5) (layer F.Cu) (net 4))
-  (segment (start 104.164 105.41) (end 101.664 102.91) (width 0.5) (layer F.Cu) (net 4))
+  (segment (start 101.664 102.91) (end 100.414 102.91) (width 0.5) (layer F.Cu) (net 4) (status 30))
+  (segment (start 108.458 105.41) (end 104.164 105.41) (width 0.5) (layer F.Cu) (net 4) (status 10))
+  (segment (start 104.164 105.41) (end 101.664 102.91) (width 0.5) (layer F.Cu) (net 4) (status 20))
   (segment (start 66.04 104.14) (end 67.379999 105.479999) (width 0.3) (layer B.Cu) (net 6) (status 10))
   (segment (start 69.93 105.49) (end 69.919999 105.479999) (width 0.5) (layer B.Cu) (net 6))
-  (segment (start 73.152 105.49) (end 69.93 105.49) (width 0.5) (layer B.Cu) (net 6))
+  (segment (start 73.152 105.49) (end 69.93 105.49) (width 0.5) (layer B.Cu) (net 6) (status 10))
   (segment (start 67.379999 105.479999) (end 69.919999 105.479999) (width 0.3) (layer B.Cu) (net 6))
   (segment (start 69.919999 105.479999) (end 71.304001 105.479999) (width 0.3) (layer B.Cu) (net 6))
   (segment (start 69.840001 100.260001) (end 69.85 100.27) (width 0.3) (layer B.Cu) (net 7))
   (segment (start 67.379999 100.260001) (end 69.840001 100.260001) (width 0.3) (layer B.Cu) (net 7))
-  (segment (start 66.04 101.6) (end 67.379999 100.260001) (width 0.3) (layer B.Cu) (net 7))
+  (segment (start 66.04 101.6) (end 67.379999 100.260001) (width 0.3) (layer B.Cu) (net 7) (status 10))
   (segment (start 70.775003 99.324999) (end 69.840001 100.260001) (width 0.5) (layer B.Cu) (net 7))
   (segment (start 77.426999 99.324999) (end 70.775003 99.324999) (width 0.5) (layer B.Cu) (net 7))
   (segment (start 77.844 99.742) (end 77.426999 99.324999) (width 0.5) (layer B.Cu) (net 7))
-  (segment (start 78.994 99.742) (end 77.844 99.742) (width 0.5) (layer B.Cu) (net 7))
-  (segment (start 75.534 102.79) (end 75.914 102.41) (width 0.5) (layer B.Cu) (net 8))
-  (segment (start 73.152 102.79) (end 75.534 102.79) (width 0.5) (layer B.Cu) (net 8))
-  (segment (start 76.962 100.41) (end 78.994 102.442) (width 0.5) (layer B.Cu) (net 9))
-  (segment (start 75.914 100.41) (end 76.962 100.41) (width 0.5) (layer B.Cu) (net 9))
+  (segment (start 78.994 99.742) (end 77.844 99.742) (width 0.5) (layer B.Cu) (net 7) (status 10))
+  (segment (start 75.532 100.41) (end 73.152 102.79) (width 0.5) (layer B.Cu) (net 8))
+  (segment (start 75.914 100.41) (end 75.532 100.41) (width 0.5) (layer B.Cu) (net 8))
+  (segment (start 75.946 102.442) (end 75.914 102.41) (width 0.5) (layer B.Cu) (net 9))
+  (segment (start 78.994 102.442) (end 75.946 102.442) (width 0.5) (layer B.Cu) (net 9))
   (via (at 101.854 104.394) (size 0.8) (drill 0.4) (layers F.Cu B.Cu) (net 10))
   (via (at 102.616 105.156) (size 0.8) (drill 0.4) (layers F.Cu B.Cu) (net 10))
