File: HB-MOD-UART-USB/HB-MOD-UART-USB.kicad_pcb (KiCad board)
At the start: 2 copper layers, 34.3 x 17.8 mm, 18 parts, among them J1 USB, Q1 IRLML6402, U1 FT232RL, U2 HM-MOD-UART

Commit message: HB-MOD-UART-USB V1.1
featuring a RX/TX LED
Parts:
- added D1: RX/TX, LEDs:LED_0603_HandSoldering, F.Cu at (133.9, 69.6)
- added R6: 270, Resistors_SMD:R_0603_HandSoldering, F.Cu at (133.9, 71.1)
Connections:
- U1 pad 23: (no net) -> Net-(D1-Pad1)
Routing:
- net Net-(D1-Pad1): track 0.00 -> 19.3 mm, vias 0 -> 2
- net +3V3: track 26.1 -> 31.7 mm
- net Net-(D1-Pad2): track 0.00 -> 1.52 mm
Other:
- board text added: "stan23 V1.1 01/2020"
- board text removed: "stan23 V1.0 01/2020"
