File: AskSinAnalyzer/AskSinAnalyzer_sheetAtmega.sch (KiCad schematic (older format))
At the start: 18 parts, among them J21 FTDI_ATmega, J22 AVR-ISP-6, U21 CC1101, U22 ATmega328PB-AU, Y21 8MHz

Commit message: PCB update
reference labels moved
Parts:
- J22: value AVR-ISP-6 -> ISP
Changed lines of the file:
@@
 P 4600 6500
 F 0 "J22" H 4321 6596 50  0000 R CNN
-F 1 "AVR-ISP-6" H 4321 6505 50  0000 R CNN
+F 1 "ISP" H 4321 6505 50  0000 R CNN
 F 2 "myPinHeaders:Pin_Header_Straight_2x03_Pitch2.54mm_Tight_Fit" V 4350 6550 50  0001 C CNN
 F 3 " ~" H 3325 5950 50  0001 C CNN

Commit message: antenna added
Parts:
- removed U21: CC1101, CC1101_Module:CC1101_Module, symbol CC1101_Module:CC1101
- added J23: Conn_Coaxial, Connectors:SMA_THT_Jack_Straight, symbol Connector:Conn_Coaxial
- added U21: CC1101, myRadioModules:CC1101_SMD_THT_Antenna, symbol myRadioModules:CC1101
- Y21: value 8MHz -> 8M; footprint myResonators:Resonator_SMD_muRata_TPSKA-3pin_7.9x3.8mm_HandSoldering -> myResonators:Resonator_SMD_muRata_CSTCC-3pin_7.2x3.0mm_HandSoldering
Connections:
- net +3V3: now also U21.1 (VCC)
- net CS: now also U21.8 (CSN)
- net GDO0: now also U21.7 (GDO0)
- net GND: now also J23.2 (Ext), U21.10 (GND), U21.11 (GND), U21.2 (GND)
- net MISO: now also U21.5 (SO)
- net MOSI: now also U21.3 (SI)
- net SCK: now also U21.4 (SCLK)
- new net: J23.1 (In), U21.9 (ANT)
- no-connect marks 19 -> 17
Other:
- note removed: "ToDo:\n- antenna"
Changed lines of the file:
@@
 $EndDescr
-$Comp
-L CC1101_Module:CC1101 U?
-U 1 1 5D4FF3D9
-P 9225 2775
-AR Path="/5D4FF3D9" Ref="U?"  Part="1"
-AR Path="/5D4E1EE1/5D4FF3D9" Ref="U21"  Part="1"
-F 0 "U21" H 9250 3464 60  0000 C CNN
-F 1 "CC1101" H 9250 3358 60  0000 C CNN
-F 2 "CC1101_Module:CC1101_Module" H 9075 3325 60  0001 C CNN
-F 3 "" H 9075 3325 60  0001 C CNN
-	1    9225 2775
-	1    0    0    -1
-$EndComp
 $Comp
 L power:GND #PWR?
@@
 Wire Wire Line
 	8725 2925 8450 2925
-NoConn ~ 9775 2625
-NoConn ~ 9775 2925
 NoConn ~ 8725 3025
 Text Label 8450 2525 0    50   ~ 0
@@
 Wire Wire Line
 	1850 6825 1850 6750
-Text Notes 8750 1675 0    100  ~ 0
-ToDo:\n- antenna
 Text HLabel 5725 3550 2    50   Input ~ 0
 ATmega_RX
@@
 P 5275 2650
 F 0 "Y21" V 5229 2761 50  0000 L CNN
-F 1 "8MHz" V 5320 2761 50  0000 L CNN
-F 2 "myResonators:Resonator_SMD_muRata_TPSKA-3pin_7.9x3.8mm_HandSoldering" H 5250 2650 50  0001 C CNN
+F 1 "8M" V 5320 2761 50  0000 L CNN
+F 2 "myResonators:Resonator_SMD_muRata_CSTCC-3pin_7.2x3.0mm_HandSoldering" H 5250 2650 50  0001 C CNN
 F 3 "~" H 5250 2650 50  0001 C CNN
 	1    5275 2650
@@
 Wire Wire Line
 	2475 1125 2475 1275
+$Comp
+L Connector:Conn_Coaxial J23
+U 1 1 5D6931D6
+P 10150 2775
+F 0 "J23" H 10250 2750 50  0000 L CNN
+F 1 "Conn_Coaxial" H 10250 2659 50  0000 L CNN
+F 2 "Connectors:SMA_THT_Jack_Straight" H 10150 2775 50  0001 C CNN
+F 3 " ~" H 10150 2775 50  0001 C CNN
+	1    10150 2775
+	1    0    0    -1
+$EndComp
+Wire Wire Line
+	9775 2775 9950 2775
+Wire Wire Line
+	9775 2625 9875 2625
+Wire Wire Line
+	9875 2625 9875 2925
+Wire Wire Line
+	9875 3025 10025 3025
+Wire Wire Line
+	10150 3025 10150 2975
+Wire Wire Line
+	9775 2925 9875 2925
+Connection ~ 9875 2925
+Wire Wire Line
+	9875 2925 9875 3025
+$Comp
+L power:GND #PWR?
+U 1 1 5D69BB80
+P 10025 3100
+AR Path="/5D69BB80" Ref="#PWR?"  Part="1"
+AR Path="/5D4E1EE1/5D69BB80" Ref="#PWR0112"  Part="1"
+F 0 "#PWR0112" H 10025 2850 50  0001 C CNN
+F 1 "GND" H 10030 2927 50  0000 C CNN
+F 2 "" H 10025 3100 50  0001 C CNN
+F 3 "" H 10025 3100 50  0001 C CNN
+	1    10025 3100
+	1    0    0    -1
+$EndComp
+Wire Wire Line
+	10025 3100 10025 3025
+Connection ~ 10025 3025
+Wire Wire Line
+	10025 3025 10150 3025
+$Comp
+L myRadioModules:CC1101 U21
+U 1 1 5D23783B
+P 9225 2775
+F 0 "U21" H 9250 3464 60  0000 C CNN
+F 1 "CC1101" H 9250 3358 60  0000 C CNN
+F 2 "myRadioModules:CC1101_SMD_THT_Antenna" H 9075 3325 60  0001 C CNN
+F 3 "" H 9075 3325 60  0001 C CNN
+	1    9225 2775
+	1    0    0    -1
+$EndComp
 $EndSCHEMATC

Commit message: AskSinAnalyzer PCB V2.0
Parts:
- removed JP21, JP22: ~, Jumper:SolderJumper-2_P1.3mm_Open_RoundedPad1.0x1.5mm, symbol Jumper:SolderJumper_2_Open
- U22: value ATmega328PB-AU -> ATmega328P-AU; symbol MCU_Microchip_ATmega:ATmega328PB-AU -> MCU_Microchip_ATmega:ATmega328P-AU
- Y21: footprint myResonators:Resonator_SMD_muRata_CSTCC-3pin_7.2x3.0mm_HandSoldering -> myResonators:Resonator_SMD_muRata_CSTCC-CSTCE-universal-3pin_7.2x3.0mm_HandSoldering
Connections:
- net RX is gone; now on net ATmega_RX: J21.3 (TX), U22.30 (PD0)
- net TX is gone; now on net ATmega_TX: J21.2 (RX), U22.31 (PD1)
- net +3V3: now also U22.6 (VCC)
- net GND: now also U22.3 (GND)
- no-connect marks 17 -> 15
Other:
- moved on the sheet: C23
Changed lines of the file:
@@
 	4725 3950 5025 3950
-$Comp
-L Jumper:SolderJumper_2_Open JP?
-U 1 1 5D4FF41F
-P 5225 3650
-AR Path="/5D4FF41F" Ref="JP?"  Part="1"
-AR Path="/5D4E1EE1/5D4FF41F" Ref="JP22"  Part="1"
-F 0 "JP22" H 5225 3550 50  0000 C CNN
-F 1 "~" H 5225 3764 50  0000 C CNN
-F 2 "Jumper:SolderJumper-2_P1.3mm_Open_RoundedPad1.0x1.5mm" H 5225 3650 50  0001 C CNN
-F 3 "~" H 5225 3650 50  0001 C CNN
-	1    5225 3650
-	1    0    0    -1
-$EndComp
-Wire Wire Line
-	4725 3650 5075 3650
-Wire Wire Line
-	5375 3650 5725 3650
 $Comp
 L Device:C C?
@@
 P 7800 2725
 AR Path="/5D4FF434" Ref="#PWR?"  Part="1"
-AR Path="/5D4E1EE1/5D4FF434" Ref="#PWR030"  Part="1"
-F 0 "#PWR030" H 7800 2475 50  0001 C CNN
+AR Path="/5D4E1EE1/5D4FF434" Ref="#PWR0123"  Part="1"
+F 0 "#PWR0123" H 7800 2475 50  0001 C CNN
 F 1 "GND" H 7805 2552 50  0000 C CNN
 F 2 "" H 7800 2725 50  0001 C CNN
@@
 Wire Wire Line
 	8200 2275 8200 2425
-$Comp
-L MCU_Microchip_ATmega:ATmega328PB-AU U?
-U 1 1 5D4FF44B
-P 4125 3050
-AR Path="/5D4FF44B" Ref="U?"  Part="1"
-AR Path="/5D4E1EE1/5D4FF44B" Ref="U22"  Part="1"
-F 0 "U22" H 3675 4500 50  0000 C CNN
-F 1 "ATmega328PB-AU" H 4025 1900 50  0000 C CNN
-F 2 "myHousings:TQFP-32_7x7mm_Pitch0.8mm_HandSoldering" H 4125 3050 50  0001 C CIN
-F 3 "http://ww1.microchip.com/downloads/en/DeviceDoc/40001906C.pdf" H 4125 3050 50  0001 C CNN
-	1    4125 3050
-	1    0    0    -1
-$EndComp
 NoConn ~ 4725 4250
 NoConn ~ 4725 4150
@@
 L Device:C C?
 U 1 1 5D4FF468
-P 3300 2050
+P 3150 2075
 AR Path="/5D4FF468" Ref="C?"  Part="1"
 AR Path="/5D4E1EE1/5D4FF468" Ref="C23"  Part="1"
-F 0 "C23" H 3415 2096 50  0000 L CNN
-F 1 "100n" H 3415 2005 50  0000 L CNN
-F 2 "Capacitors_SMD:C_0805_HandSoldering" H 3338 1900 50  0001 C CNN
-F 3 "~" H 3300 2050 50  0001 C CNN
-	1    3300 2050
-	1    0    0    -1
-$EndComp
-Wire Wire Line
-	3300 1900 3300 1850
-Wire Wire Line
-	3300 1850 3525 1850
+F 0 "C23" H 3265 2121 50  0000 L CNN
+F 1 "100n" H 3265 2030 50  0000 L CNN
+F 2 "Capacitors_SMD:C_0805_HandSoldering" H 3188 1925 50  0001 C CNN
+F 3 "~" H 3150 2075 50  0001 C CNN
+	1    3150 2075
+	1    0    0    -1
+$EndComp
+Wire Wire Line
+	3150 1925 3150 1850
+Wire Wire Line
+	3150 1850 3525 1850
 $Comp
 L power:GND #PWR?
 U 1 1 5D4FF470
-P 3300 2300
+P 3150 2300
 AR Path="/5D4FF470" Ref="#PWR?"  Part="1"
 AR Path="/5D4E1EE1/5D4FF470" Ref="#PWR0105"  Part="1"
-F 0 "#PWR0105" H 3300 2050 50  0001 C CNN
-F 1 "GND" H 3305 2127 50  0000 C CNN
-F 2 "" H 3300 2300 50  0001 C CNN
-F 3 "" H 3300 2300 50  0001 C CNN
-	1    3300 2300
+F 0 "#PWR0105" H 3150 2050 50  0001 C CNN
+F 1 "GND" H 3155 2127 50  0000 C CNN
+F 2 "" H 3150 2300 50  0001 C CNN
+F 3 "" H 3150 2300 50  0001 C CNN
+	1    3150 2300
 	1    0    0    -1
 $EndComp
@@
 Wire Wire Line
 	4125 4625 4125 4550
-NoConn ~ 3525 3550
-NoConn ~ 3525 3650
-NoConn ~ 3525 3750
-NoConn ~ 3525 3850
 Text Label 5025 3650 2    50   ~ 0
 TX
-$Comp
-L Jumper:SolderJumper_2_Open JP?
-U 1 1 5D4FF482
-P 5225 3550
-AR Path="/5D4FF482" Ref="JP?"  Part="1"
-AR Path="/5D4E1EE1/5D4FF482" Ref="JP21"  Part="1"
-F 0 "JP21" H 5225 3650 50  0000 C CNN
-F 1 "~" H 5225 3664 50  0000 C CNN
-F 2 "Jumper:SolderJumper-2_P1.3mm_Open_RoundedPad1.0x1.5mm" H 5225 3550 50  0001 C CNN
-F 3 "~" H 5225 3550 50  0001 C CNN
-	1    5225 3550
-	1    0    0    -1
-$EndComp
-Wire Wire Line
-	4725 3550 5075 3550
-Wire Wire Line
-	5375 3550 5725 3550
-Wire Wire Line
-	3300 2300 3300 2200
+Wire Wire Line
+	3150 2300 3150 2225
 $Comp
 L myConnectors:FtdiConnector J?
@@
 Wire Wire Line
 	1850 6825 1850 6750
-Text HLabel 5725 3550 2    50   Input ~ 0
+Text HLabel 5175 3550 2    50   Input ~ 0
 ATmega_RX
-Text HLabel 5725 3650 2    50   Input ~ 0
+Text HLabel 5175 3650 2    50   Input ~ 0
 ATmega_TX
-$Comp
-L Device:Resonator Y21
-U 1 1 5D5D1C09
-P 5275 2650
-F 0 "Y21" V 5229 2761 50  0000 L CNN
-F 1 "8M" V 5320 2761 50  0000 L CNN
-F 2 "myResonators:Resonator_SMD_muRata_CSTCC-3pin_7.2x3.0mm_HandSoldering" H 5250 2650 50  0001 C CNN
-F 3 "~" H 5250 2650 50  0001 C CNN
-	1    5275 2650
-	0    -1   1    0
-$EndComp
-$Comp
-L Device:R R?
-U 1 1 5D5D985A
-P 5725 2650
-AR Path="/5D5D985A" Ref="R?"  Part="1"
-AR Path="/5D4E1EE1/5D5D985A" Ref="R22"  Part="1"
-F 0 "R22" H 5795 2696 50  0000 L CNN
-F 1 "1M" H 5795 2605 50  0000 L CNN
-F 2 "Resistors_SMD:R_0805_HandSoldering" V 5655 2650 50  0001 C CNN
-F 3 "~" H 5725 2650 50  0001 C CNN
-	1    5725 2650
-	1    0    0    -1
-$EndComp
-Wire Wire Line
-	4725 2450 5275 2450
-Wire Wire Line
-	5275 2500 5275 2450
-Connection ~ 5275 2450
-Wire Wire Line
-	5275 2450 5725 2450
-Wire Wire Line
-	5725 2500 5725 2450
-Wire Wire Line
-	5725 2800 5725 2850
-Wire Wire Line
-	5725 2850 5275 2850
-Wire Wire Line
-	5275 2850 5275 2800
-Wire Wire Line
-	5275 2850 4925 2850
 Wire Wire Line
 	4925 2850 4925 2550
 Wire Wire Line
 	4925 2550 4725 2550
-Connection ~ 5275 2850
-$Comp
-L power:GND #PWR?
-U 1 1 5D5DF898
-P 5525 2925
-AR Path="/5D5DF898" Ref="#PWR?"  Part="1"
-AR Path="/5D4E1EE1/5D5DF898" Ref="#PWR031"  Part="1"
-F 0 "#PWR031" H 5525 2675 50  0001 C CNN
-F 1 "GND" H 5530 2752 50  0000 C CNN
-F 2 "" H 5525 2925 50  0001 C CNN
-F 3 "" H 5525 2925 50  0001 C CNN
-	1    5525 2925
-	1    0    0    -1
-$EndComp
-Wire Wire Line
-	5525 2925 5525 2650
-Wire Wire Line
-	5525 2650 5475 2650
 Wire Wire Line
 	1850 6075 1850 6100
@@
 	1    0    0    -1
 $EndComp
+$Comp
+L MCU_Microchip_ATmega:ATmega328P-AU U?
+U 1 1 5D4FF44B
+P 4125 3050
+AR Path="/5D4FF44B" Ref="U?"  Part="1"
+AR Path="/5D4E1EE1/5D4FF44B" Ref="U22"  Part="1"
+F 0 "U22" H 3675 4500 50  0000 C CNN
+F 1 "ATmega328P-AU" H 4025 1900 50  0000 C CNN
+F 2 "myHousings:TQFP-32_7x7mm_Pitch0.8mm_HandSoldering" H 4125 3050 50  0001 C CIN
+F 3 "http://ww1.microchip.com/downloads/en/DeviceDoc/40001906C.pdf" H 4125 3050 50  0001 C CNN
+	1    4125 3050
+	1    0    0    -1
+$EndComp
+NoConn ~ 3525 2050
+NoConn ~ 3525 2150
+Wire Wire Line
+	5275 2850 4925 2850
+Connection ~ 5275 2850
+Wire Wire Line
+	5275 2850 5275 2800
+Wire Wire Line
+	4725 2450 5275 2450
+Connection ~ 5275 2450
+Wire Wire Line
+	5275 2500 5275 2450
+Wire Wire Line
+	5275 2450 5725 2450
+Wire Wire Line
+	5725 2500 5725 2450
+Wire Wire Line
+	5725 2800 5725 2850
+Wire Wire Line
+	5725 2850 5275 2850
+$Comp
+L power:GND #PWR?
+U 1 1 5D5DF898
+P 5525 2925
+AR Path="/5D5DF898" Ref="#PWR?"  Part="1"
+AR Path="/5D4E1EE1/5D5DF898" Ref="#PWR031"  Part="1"
+F 0 "#PWR031" H 5525 2675 50  0001 C CNN
+F 1 "GND" H 5530 2752 50  0000 C CNN
+F 2 "" H 5525 2925 50  0001 C CNN
+F 3 "" H 5525 2925 50  0001 C CNN
+	1    5525 2925
+	1    0    0    -1
+$EndComp
+Wire Wire Line
+	5525 2650 5475 2650
+Wire Wire Line
+	5525 2925 5525 2650
+$Comp
+L Device:Resonator Y21
+U 1 1 5D5D1C09
+P 5275 2650
+F 0 "Y21" V 5229 2761 50  0000 L CNN
+F 1 "8M" V 5320 2761 50  0000 L CNN
+F 2 "myResonators:Resonator_SMD_muRata_CSTCC-CSTCE-universal-3pin_7.2x3.0mm_HandSoldering" H 5250 2650 50  0001 C CNN
+F 3 "~" H 5250 2650 50  0001 C CNN
+	1    5275 2650
+	0    -1   1    0
+$EndComp
+$Comp
+L Device:R R?
+U 1 1 5D5D985A
+P 5725 2650
+AR Path="/5D5D985A" Ref="R?"  Part="1"
+AR Path="/5D4E1EE1/5D5D985A" Ref="R22"  Part="1"
+F 0 "R22" H 5795 2696 50  0000 L CNN
+F 1 "1M" H 5795 2605 50  0000 L CNN
+F 2 "Resistors_SMD:R_0805_HandSoldering" V 5655 2650 50  0001 C CNN
+F 3 "~" H 5725 2650 50  0001 C CNN
+	1    5725 2650
+	1    0    0    -1
+$EndComp
+Wire Wire Line
+	4725 3650 5175 3650
+Wire Wire Line
+	4725 3550 5175 3550
 $EndSCHEMATC

Commit message: add production data to AskSinAnalyzer PCB
Parts:
- C21: LCSC (none) -> C15850
- C22, C23, C25, C26: LCSC (none) -> C49678
- C24: LCSC (none) -> C28323
- J21, J22, J23, LED21, U21: LCSC (none) -> -
- R21, R23: LCSC (none) -> C17414
- R22: LCSC (none) -> C17514
- R24: LCSC (none) -> C17630
- U22: LCSC (none) -> C14877
Changed lines of the file:
@@
 F 2 "Resistors_SMD:R_0805_HandSoldering" V 7205 5425 50  0001 C CNN
 F 3 "~" H 7275 5425 50  0001 C CNN
+F 4 "C17630" H 7275 5425 50  0001 C CNN "LCSC"
 	1    7275 5425
 	0    1    1    0
@@
 F 2 "LEDs:LED_D3.0mm_Horizontal_O3.81mm_Z6.0mm" H 7700 5425 50  0001 C CNN
 F 3 "~" H 7700 5425 50  0001 C CNN
+F 4 "-" H 7700 5425 50  0001 C CNN "LCSC"
 	1    7700 5425
 	-1   0    0    1
@@
 F 2 "Capacitors_SMD:C_0805_HandSoldering" H 7838 2350 50  0001 C CNN
 F 3 "~" H 7800 2500 50  0001 C CNN
+F 4 "C28323" H 7800 2500 50  0001 C CNN "LCSC"
 	1    7800 2500
 	1    0    0    -1
@@
 F 2 "Resistors_SMD:R_0805_HandSoldering" V 8130 2575 50  0001 C CNN
 F 3 "~" H 8200 2575 50  0001 C CNN
+F 4 "C17414" H 8200 2575 50  0001 C CNN "LCSC"
 	1    8200 2575
 	1    0    0    -1
@@
 F 2 "Capacitors_SMD:C_0805_HandSoldering" H 3188 1925 50  0001 C CNN
 F 3 "~" H 3150 2075 50  0001 C CNN
+F 4 "C49678" H 3150 2075 50  0001 C CNN "LCSC"
 	1    3150 2075
 	1    0    0    -1
@@
 F 2 "myPinHeaders:Pin_Header_Straight_1x06_Pitch2.54mm_Tight_Fit" H 1925 6450 50  0001 C CNN
 F 3 "" H 1925 6450 50  0001 C CNN
+F 4 "-" H 1925 6450 50  0001 C CNN "LCSC"
 	1    1925 6450
 	1    0    0    -1
@@
 F 2 "myPinHeaders:Pin_Header_Straight_2x03_Pitch2.54mm_Tight_Fit" V 4350 6550 50  0001 C CNN
 F 3 " ~" H 3325 5950 50  0001 C CNN
+F 4 "-" H 4600 6500 50  0001 C CNN "LCSC"
 	1    4600 6500
 	1    0    0    -1
@@
 F 2 "Capacitors_SMD:C_0805_HandSoldering" H 1713 5200 50  0001 C CNN
 F 3 "~" H 1675 5350 50  0001 C CNN
+F 4 "C49678" H 1675 5350 50  0001 C CNN "LCSC"
 	1    1675 5350
 	0    1    1    0
@@
 F 2 "Resistors_SMD:R_0805_HandSoldering" V 2055 5100 50  0001 C CNN
 F 3 "~" H 2125 5100 50  0001 C CNN
+F 4 "C17414" H 2125 5100 50  0001 C CNN "LCSC"
 	1    2125 5100
 	-1   0    0    1
@@
 F 2 "Capacitors_SMD:C_0805_HandSoldering" H 2038 1275 50  0001 C CNN
 F 3 "~" H 2000 1425 50  0001 C CNN
+F 4 "C49678" H 2000 1425 50  0001 C CNN "LCSC"
 	1    2000 1425
 	1    0    0    -1
@@
 F 2 "Capacitors_SMD:C_0805_HandSoldering" H 1588 1275 50  0001 C CNN
 F 3 "~" H 1550 1425 50  0001 C CNN
+F 4 "C15850" H 1550 1425 50  0001 C CNN "LCSC"
 	1    1550 1425
 	1    0    0    -1
@@
 F 2 "Capacitors_SMD:C_0805_HandSoldering" H 2513 1275 50  0001 C CNN
 F 3 "~" H 2475 1425 50  0001 C CNN
+F 4 "C49678" H 2475 1425 50  0001 C CNN "LCSC"
 	1    2475 1425
 	1    0    0    -1
@@
 F 2 "Connectors:SMA_THT_Jack_Straight" H 10150 2775 50  0001 C CNN
 F 3 " ~" H 10150 2775 50  0001 C CNN
+F 4 "-" H 10150 2775 50  0001 C CNN "LCSC"
 	1    10150 2775
 	1    0    0    -1
@@
 F 2 "myRadioModules:CC1101_SMD_THT_Antenna" H 9075 3325 60  0001 C CNN
 F 3 "" H 9075 3325 60  0001 C CNN
+F 4 "-" H 9225 2775 50  0001 C CNN "LCSC"
 	1    9225 2775
 	1    0    0    -1
@@
 F 2 "myHousings:TQFP-32_7x7mm_Pitch0.8mm_HandSoldering" H 4125 3050 50  0001 C CIN
 F 3 "http://ww1.microchip.com/downloads/en/DeviceDoc/40001906C.pdf" H 4125 3050 50  0001 C CNN
+F 4 "C14877" H 4125 3050 50  0001 C CNN "LCSC"
 	1    4125 3050
 	1    0    0    -1
@@
 F 2 "Resistors_SMD:R_0805_HandSoldering" V 5655 2650 50  0001 C CNN
 F 3 "~" H 5725 2650 50  0001 C CNN
+F 4 "C17514" H 5725 2650 50  0001 C CNN "LCSC"
 	1    5725 2650
 	1    0    0    -1
