File: HB-LC-Dim5PWM-CV_AskSinDuino32Shield/HB-LC-Dim5PWM-CV_AskSinDuino32Shield.kicad_sch (KiCad schematic)
At the start: 35 parts, among them J1 power+LED, J2 Encoder 1, J3 Encoder 2, Q11 IRF3708, Q12 IRF3708, Q13 IRF3708, Q14 IRF3708, U1 AskSinDuino32, U2 DS18B20, U3 LC78_05-0.5

Commit message: HB-LC-Dim5PWM-CV_AskSinDuino32Shield
- 5th channel
- SMD FETs
- mounting holes
- PCB size and routing optimized
Parts:
- removed D1, D2, D3, D4: SS16, Diode_SMD:D_SMA, symbol Device:D
- removed Q11, Q12, Q13, Q14: IRF3708, Package_TO_SOT_THT:TO-220-3_Vertical, symbol Simulation_SPICE:NMOS
- added H1: MountingHole, MountingHole:MountingHole_3.2mm_M3, symbol Mechanical:MountingHole
- added H2: MountingHole, MountingHole:MountingHole_3.5mm, symbol Mechanical:MountingHole
- added Q11, Q12, Q13, Q14, Q15: IRF8788PbF, Package_SO:SOIC-8_3.9x4.9mm_P1.27mm, symbol Transistor_FET:IRF8721PBF-1
- added R19: 100R, Resistor_SMD:R_0805_2012Metric_Pad1.20x1.40mm_HandSolder, symbol Device:R
- added R20: 100k, Resistor_SMD:R_0805_2012Metric_Pad1.20x1.40mm_HandSolder, symbol Device:R
Connections:
- net +24V: now also J1.7 (Pin_7); no longer J1.5 (Pin_5)
- net 1WIRE: now also U1.W12 (PA1); no longer U1.W11 (PA2)
- net GND: now also Q11.1 (S), Q11.2 (S), Q11.3 (S), Q12.1 (S), Q12.2 (S), Q12.3 (S), Q13.1 (S), Q13.2 (S), Q13.3 (S), Q14.1 (S), Q14.2 (S), Q14.3 (S), Q15.1 (S), Q15.2 (S), Q15.3 (S), R20.1; no longer J1.7 (Pin_7)
- net LED1: now also J1.5 (Pin_5), Q11.5 (D), Q11.6 (D), Q11.7 (D), Q11.8 (D); no longer J1.1 (Pin_1)
- net LED2: now also J1.4 (Pin_4), Q12.5 (D), Q12.6 (D), Q12.7 (D), Q12.8 (D); no longer J1.2 (Pin_2)
- net LED3: now also Q13.5 (D), Q13.6 (D), Q13.7 (D), Q13.8 (D)
- net LED4: now also J1.2 (Pin_2), Q14.5 (D), Q14.6 (D), Q14.7 (D), Q14.8 (D); no longer J1.4 (Pin_4)
- net PWM1: now also U1.W8 (PA5); no longer U1.W6 (PA7)
- net PWM3: now also U1.W6 (PA7); no longer U1.W8 (PA5)
- net PWM4: now also U1.W5 (PB0); no longer U1.W9 (PA4)
- net at R17.2, R18.2: now also Q14.4 (G)
- net at R13.2, R14.2: now also Q12.4 (G)
- net at R11.2, R12.2: now also Q11.4 (G)
- net at R15.2, R16.2: now also Q13.4 (G)
- net PWM5: now reaches U1.W4 (PB1)
- net PWM5: now also R19.1
- new net: Q15.4 (G), R19.2, R20.2
- new net LED5: J1.1 (Pin_1), Q15.5 (D), Q15.6 (D), Q15.7 (D), Q15.8 (D)
- no-connect marks 17 -> 16
